File: il2450_ElectronicSystemsDesign/il2450_lab1.sch (KiCad schematic (older format))
At the start: 21 parts, among them P1 USB_OTG, P2 Spy-Bi-Wire, P3 UART, U1 LM1117-3.3, U2 MSP430G2553IPW20, U3 TMP101NA/250, Y1 Crystal

Commit message: Some more exports
Parts:
- D1: value LED -> GREEN
- D2: value LED -> RED
- U2: value MSP430G2553IPW20 -> MSP430G2553; Details (none) -> TSSOP-20
- Y1: value Crystal -> 12 MHz
Changed lines of the file:
@@
 P 4750 4650
 F 0 "U2" H 3250 5250 50  0000 C CNN
-F 1 "MSP430G2553IPW20" H 6000 4100 50  0000 C CNN
+F 1 "MSP430G2553" H 6000 4100 50  0000 C CNN
 F 2 "Housings_SSOP:TSSOP-20_4.4x6.5mm_Pitch0.65mm" H 3300 4100 50  0001 C CIN
 F 3 "" H 4700 4650 50  0000 C CNN
+F 4 "TSSOP-20" H 4750 4650 60  0001 C CNN "Details"
 	1    4750 4650
 	1    0    0    -1
@@
 P 2600 5000
 F 0 "Y1" H 2600 5150 50  0000 C CNN
-F 1 "Crystal" H 2600 4850 50  0000 C CNN
+F 1 "12 MHz" H 2600 4850 50  0000 C CNN
 F 2 "Crystals:Crystal_SMD_HC49-SD" H 2600 5000 50  0001 C CNN
 F 3 "" H 2600 5000 50  0000 C CNN
@@
 P 1450 4750
 F 0 "D1" H 1450 4850 50  0000 C CNN
-F 1 "LED" H 1450 4650 50  0000 C CNN
+F 1 "GREEN" H 1450 4650 50  0000 C CNN
 F 2 "LEDs:LED_0805" H 1450 4750 50  0001 C CNN
 F 3 "" H 1450 4750 50  0000 C CNN
@@
 P 1850 4750
 F 0 "D2" H 1850 4850 50  0000 C CNN
-F 1 "LED" H 1850 4650 50  0000 C CNN
+F 1 "RED" H 1850 4650 50  0000 C CNN
 F 2 "LEDs:LED_0805" H 1850 4750 50  0001 C CNN
 F 3 "" H 1850 4750 50  0000 C CNN
